Commit message: added stir_bringup

File: ros/stir_description/robot/crane_x7_with_tools.urdf.xacro (robot description, xacro)
@@ -1,19 +1,18 @@
 <?xml version="1.0"?>
-<robot name="stir"
+<!-- TODO(sara): rename robot name to crane_x7_with_tools -->
+<robot name="crane_x7"
        xmlns:xacro="http://ros.org/wiki/xacro"
        xmlns:sensor="http://playerstage.sourceforge.net/gazebo/xmlschema/#sensor"
        xmlns:controller="http://playerstage.sourceforge.net/gazebo/xmlschema/#controller"
        xmlns:interface="http://playerstage.sourceforge.net/gazebo/xmlschema/#interface">
+  <xacro:include filename="$(find crane_x7_description)/urdf/crane_x7.xacro" />
+  <link name="base_link" />
   <link name="world" />
-  <link name="crane_x7_base_link" />
-  <xacro:property name="crane_x7_base_x" value="-0.3" />
-  <joint name="crane_x7_base_link_to_world_joint" type="fixed">
-    <origin xyz="${crane_x7_base_x} 0 0" rpy="0 0 0"/>
-    <parent link="world"/>="-
-    <child link="crane_x7_base_link"/>
+  <joint name="base_link_to_world_joint" type="fixed">
+    <parent link="world"/>
+    <child link="base_link"/>
   </joint>
   <xacro:arg name="use_effort_gripper" default="false" />
-  <xacro:include filename="$(find crane_x7_description)/urdf/crane_x7.xacro"/>
-  <xacro:crane_x7 parent="crane_x7_base_link"
+  <xacro:crane_x7 parent="base_link"
                   base_color="red"
                   shoulder_color="white"
@@ -39,9 +38,7 @@
   <xacro:property name="tool_orientation_p" value="0.02" />
   <xacro:property name="tool_end_position_z" value="0.35" />
-  <xacro:property name="ingredients_position_z" value="0.1" />
-  <xacro:property name="ingredients_radius" value="0.01" />
   <link name="tool_link">
     <visual>
-      <origin rpy="0 ${tool_orientation_p} 0" xyz="${tool_position_x} 0 -${tool_position_z}"/>
+      <origin rpy="0 -${tool_orientation_p} 0" xyz="${tool_position_x} 0 -${tool_position_z}"/>
       <geometry>
         <cylinder radius="${tool_radius}" length="${tool_length}"/>
@@ -49,29 +46,26 @@
     </visual>
     <visual>
-      <origin rpy="0 -${tool_orientation_p} 0" xyz="-${tool_position_x} 0 -${tool_position_z}"/>
+      <origin rpy="0 ${tool_orientation_p} 0" xyz="-${tool_position_x} 0 -${tool_position_z}"/>
       <geometry>
         <cylinder radius="${tool_radius}" length="${tool_length}"/>
       </geometry>
     </visual>
+    <collision>
+      <origin rpy="0 -${tool_orientation_p} 0" xyz="${tool_position_x} 0 -${tool_position_z}"/>
+      <geometry>
+        <cylinder radius="${tool_radius}" length="${tool_length}"/>
+      </geometry>
+    </collision>
+    <collision>
+      <origin rpy="0 ${tool_orientation_p} 0" xyz="-${tool_position_x} 0 -${tool_position_z}"/>
+      <geometry>
+        <cylinder radius="${tool_radius}" length="${tool_length}"/>
+      </geometry>
+    </collision>
   </link>
-  <joint name="tool_link_to_gripper_base_link" type="fixed">
+  <joint name="tool_link_to_gripper_base_joint" type="fixed">
     <origin rpy="0 0 0" xyz="0 0 ${tool_end_position_z}"/>
     <parent link="crane_x7_gripper_base_link" />
     <child link="tool_link" />
   </joint>
-  <link name="bowl_link">
-    <visual>
-      <origin xyz="0 0 0" rpy="0 0 0"/>
-      <geometry>
-        <mesh filename="package://stir_description/meshes/bowl5.stl"/>
-      </geometry>
-      <material name="clear">
-        <color rgba="0.8 0.8 0.8 0.8"/>
-      </material>
-    </visual>
-  </link>
-  <joint name="bowl_link_to_world" type="fixed">
-    <parent link="world" />
-    <child link="bowl_link" />
-  </joint>
 </robot>

Commit message: changed tools position to ignore collision

File: ros/stir_description/robot/crane_x7_with_tools.urdf.xacro (robot description, xacro)
@@ -13,5 +13,5 @@
     <child link="base_link"/>
   </joint>
-  <xacro:arg name="use_effort_gripper" default="false" />
+  <xacro:arg name="use_effort_gripper" default="true" />
   <xacro:crane_x7 parent="base_link"
                   base_color="red"
@@ -37,5 +37,6 @@
   <xacro:property name="tool_position_z" value="${tool_length/2}" />
   <xacro:property name="tool_orientation_p" value="0.02" />
-  <xacro:property name="tool_end_position_z" value="0.35" />
+  <!-- TODO(sara): resolve collision probrem -->
+  <xacro:property name="tool_end_position_z" value="0.39" />
   <link name="tool_link">
     <visual>

Commit message: tain with ingredients using gazebo

File: ros/stir_description/robot/crane_x7_with_tools.urdf.xacro (robot description, xacro)
@@ -32,11 +32,11 @@
     <origin xyz="0 0 0"/>
   </xacro:crane_x7>
-  <xacro:property name="tool_length" value="0.3" />
-  <xacro:property name="tool_radius" value="0.003" />
-  <xacro:property name="tool_position_x" value="0.01" />
+  <xacro:property name="tool_length" value="0.27" />
+  <xacro:property name="tool_radius" value="0.002" />
+  <xacro:property name="tool_position_x" value="0.012" />
   <xacro:property name="tool_position_z" value="${tool_length/2}" />
-  <xacro:property name="tool_orientation_p" value="0.02" />
+  <xacro:property name="tool_orientation_p" value="0.05" />
   <!-- TODO(sara): resolve collision probrem -->
-  <xacro:property name="tool_end_position_z" value="0.39" />
+  <xacro:property name="tool_end_position_z" value="0.325" />
   <link name="tool_link">
     <visual>

Commit message: added tools.xacro

File: ros/stir_description/robot/crane_x7_with_tools.urdf.xacro (robot description, xacro)
@@ -1,5 +1,4 @@
 <?xml version="1.0"?>
-<!-- TODO(sara): rename robot name to crane_x7_with_tools -->
-<robot name="crane_x7"
+<robot name="crane_x7_with_tools"
        xmlns:xacro="http://ros.org/wiki/xacro"
        xmlns:sensor="http://playerstage.sourceforge.net/gazebo/xmlschema/#sensor"
@@ -7,4 +6,5 @@
        xmlns:interface="http://playerstage.sourceforge.net/gazebo/xmlschema/#interface">
   <xacro:include filename="$(find crane_x7_description)/urdf/crane_x7.xacro" />
+  <xacro:include filename="$(find stir_description)/robot/tools.xacro" />
   <link name="base_link" />
   <link name="world" />
@@ -32,41 +32,4 @@
     <origin xyz="0 0 0"/>
   </xacro:crane_x7>
-  <xacro:property name="tool_length" value="0.27" />
-  <xacro:property name="tool_radius" value="0.002" />
-  <xacro:property name="tool_position_x" value="0.012" />
-  <xacro:property name="tool_position_z" value="${tool_length/2}" />
-  <xacro:property name="tool_orientation_p" value="0.05" />
-  <!-- TODO(sara): resolve collision probrem -->
-  <xacro:property name="tool_end_position_z" value="0.325" />
-  <link name="tool_link">
-    <visual>
-      <origin rpy="0 -${tool_orientation_p} 0" xyz="${tool_position_x} 0 -${tool_position_z}"/>
-      <geometry>
-        <cylinder radius="${tool_radius}" length="${tool_length}"/>
-      </geometry>
-    </visual>
-    <visual>
-      <origin rpy="0 ${tool_orientation_p} 0" xyz="-${tool_position_x} 0 -${tool_position_z}"/>
-      <geometry>
-        <cylinder radius="${tool_radius}" length="${tool_length}"/>
-      </geometry>
-    </visual>
-    <collision>
-      <origin rpy="0 -${tool_orientation_p} 0" xyz="${tool_position_x} 0 -${tool_position_z}"/>
-      <geometry>
-        <cylinder radius="${tool_radius}" length="${tool_length}"/>
-      </geometry>
-    </collision>
-    <collision>
-      <origin rpy="0 ${tool_orientation_p} 0" xyz="-${tool_position_x} 0 -${tool_position_z}"/>
-      <geometry>
-        <cylinder radius="${tool_radius}" length="${tool_length}"/>
-      </geometry>
-    </collision>
-  </link>
-  <joint name="tool_link_to_gripper_base_joint" type="fixed">
-    <origin rpy="0 0 0" xyz="0 0 ${tool_end_position_z}"/>
-    <parent link="crane_x7_gripper_base_link" />
-    <child link="tool_link" />
-  </joint>
+  <xacro:tools />
 </robot>
